Commit message: The basic navigation model (differential style type) seems to work properly now

File: visualiser/robot_models/four_wheel.urdf (robot description, URDF)
Before this commit: robot robot, 5 links, 4 joints
Links:
- added link laser_scanner; visual box size=0.1 0.2 0.1
Joints:
- added joint joint_laser_scanner: type continuous, parent base_link, child laser_scanner, origin xyz=0.45 0.0 0.175 rpy=0 0 0, axis 0 1 0

Commit message: Added a node that simulates laser scans, though I currently have some mistake in the calculations of the scans

File: visualiser/robot_models/four_wheel.urdf (robot description, URDF)
Before this commit: robot robot, 6 links, 5 joints
Links:
- removed link laser_scanner
- added link laser_front; visual box size=0.1 0.05 0.05
- added link laser_front_left; visual box size=0.1 0.05 0.05
- added link laser_front_right; visual box size=0.1 0.05 0.05
- added link laser_left; visual box size=0.1 0.05 0.05
- added link laser_right; visual box size=0.1 0.05 0.05
Joints:
- removed joint joint_laser_scanner
- added joint joint_laser_front: type continuous, parent base_link, child laser_front, origin xyz=0.45 0.0 0.15 rpy=0 0 0, axis 0 1 0
- added joint joint_laser_front_left: type continuous, parent base_link, child laser_front_left, origin xyz=0.45 0.2 0.15 rpy=0 0 0.785398, axis 0 1 0
- added joint joint_laser_front_right: type continuous, parent base_link, child laser_front_right, origin xyz=0.45 -0.2 0.15 rpy=0 0 -0.785398, axis 0 1 0
- added joint joint_laser_left: type continuous, parent base_link, child laser_left, origin xyz=0 0.2 0.15 rpy=0 0 1.57070796, axis 0 1 0
- added joint joint_laser_right: type continuous, parent base_link, child laser_right, origin xyz=0 -0.2 0.15 rpy=0 0 -1.57070796, axis 0 1 0

Commit message: Made some progress with the laser scanner, though I'm currently getting incorrect measurements when the robot is moving

File: visualiser/robot_models/four_wheel.urdf (robot description, URDF)
Before this commit: robot robot, 10 links, 9 joints
Links:
- removed link laser_front_left
- removed link laser_front_right
- removed link laser_left
- removed link laser_right
- link laser_front: geometry visual box size=0.05 0.1 0.05
Joints:
- removed joint joint_laser_front_left
- removed joint joint_laser_front_right
- removed joint joint_laser_left
- removed joint joint_laser_right
- joint joint_laser_front: origin xyz=0.45 0.0 0.15 rpy=0 0 0 -> xyz=0.475 0.0 0.15 rpy=0 0 0

Commit message: Added a back laser scanner in addition to the front one

File: visualiser/robot_models/four_wheel.urdf (robot description, URDF)
Before this commit: robot robot, 6 links, 5 joints
Links:
- added link front_marker; visual box size=0.01 0.5 0.25
- added link laser_back; visual box size=0.05 0.1 0.05
Joints:
- added joint joint_front_marker: type continuous, parent base_link, child front_marker, origin xyz=0.5 0 0 rpy=0 0 0, axis 0 1 0
- added joint joint_laser_back: type continuous, parent base_link, child laser_back, origin xyz=-0.475 0.0 0.15 rpy=0 0 3.14, axis 0 1 0
